Commit message: Gazebo is working properly need to add world frame and some gazebo puglins

File: urdf/arm_controller.xacro (robot description, xacro)
@@ -1,8 +1,103 @@
 <?xml version="1.0" ?>
 <robot name="cycloidal_arm" xmlns:xacro="http://www.ros.org/wiki/xacro" >
+<ros2_control name="GazeboSystem" type="system">
+    <hardware>
+        <plugin>gazebo_ros2_control/GazeboSystem</plugin>
+    </hardware>
+    <joint name="Revolute_1">
+        <command_interface name="position">
+            <param name="min">-10</param>
+            <param name="max">10</param>
+        </command_interface>
+        <state_interface name="position"/>
+        <state_interface name="velocity"/>
+        <state_interface name="effort"/>
+    </joint>
+    <joint name="Revolute_2">
+        <command_interface name="position">
+            <param name="min">-10</param>
+            <param name="max">10</param>
+        </command_interface>
+        <state_interface name="position"/>
+        <state_interface name="velocity"/>
+        <state_interface name="effort"/>
+    </joint>
+    <joint name="Revolute_3">
+        <command_interface name="position">
+            <param name="min">-10</param>
+            <param name="max">10</param>
+        </command_interface>
+        <state_interface name="position"/>
+        <state_interface name="velocity"/>
+        <state_interface name="effort"/>
+    </joint>
+    <joint name="Revolute_4">
+        <command_interface name="position">
+            <param name="min">-10</param>
+            <param name="max">10</param>
+        </command_interface>
+        <state_interface name="position"/>
+        <state_interface name="velocity"/>
+        <state_interface name="effort"/>
+    </joint>
+    <joint name="Revolute_5">
+        <command_interface name="position">
+            <param name="min">-10</param>
+            <param name="max">10</param>
+        </command_interface>
+        <state_interface name="position"/>
+        <state_interface name="velocity"/>
+        <state_interface name="effort"/>
+    </joint>
+</ros2_control>
 <gazebo>
     <puglin name="gazebo_ros2_control" filename="libgazebo_ros2_control.so">
-        <parameters></parameters>
+        <robot_sim_type>gazebo_ros2_control/GazeboSystem</robot_sim_type>
+        <parameters>$(find cycloidal_arm)/config/my_controller.yaml</parameters>
     </puglin>
 </gazebo>
+<xacro:property name="body_color" value="Gazebo/Silver" />
+<gazebo reference="base_link">
+  <material>${body_color}</material>
+  <mu1>0.2</mu1>
+  <mu2>0.2</mu2>
+  <selfCollide>true</selfCollide>
+  <gravity>true</gravity>
+</gazebo>
+<gazebo reference="link_1_1">
+  <material>${body_color}</material>
+  <mu1>0.2</mu1>
+  <mu2>0.2</mu2>
+  <selfCollide>true</selfCollide>
+</gazebo>
+<gazebo reference="link_2_1">
+  <material>${body_color}</material>
+  <mu1>0.2</mu1>
+  <mu2>0.2</mu2>
+  <selfCollide>true</selfCollide>
+</gazebo>
+<gazebo reference="link_3_1">
+  <material>${body_color}</material>
+  <mu1>0.2</mu1>
+  <mu2>0.2</mu2>
+  <selfCollide>true</selfCollide>
+</gazebo>
+<gazebo reference="link_4_1">
+  <material>${body_color}</material>
+  <mu1>0.2</mu1>
+  <mu2>0.2</mu2>
+  <selfCollide>true</selfCollide>
+</gazebo>
+<gazebo reference="link_5_1">
+  <material>${body_color}</material>
+  <mu1>0.2</mu1>
+  <mu2>0.2</mu2>
+  <selfCollide>true</selfCollide>
+</gazebo>
+<gazebo reference="camera_1">
+  <material>${body_color}</material>
+  <mu1>0.2</mu1>
+  <mu2>0.2</mu2>
+  <selfCollide>true</selfCollide>
+</gazebo>
 </robot>

File: urdf/cycloidal_arm.xacro (robot description, xacro)
@@ -11,5 +11,5 @@
     <origin xyz="0 0 0" rpy="0 0 0"/>
     <geometry>
-      <mesh filename="package://cycloidal_arm/meshes/base_link.stl" scale="0.001 0.001 0.001"/>
+      <mesh filename="file://$(find cycloidal_arm)/meshes/base_link.stl" scale="0.001 0.001 0.001"/>
     </geometry>
     <material name="silver"/>
@@ -18,18 +18,18 @@
     <origin xyz="0 0 0" rpy="0 0 0"/>
     <geometry>
-      <mesh filename="package://cycloidal_arm/meshes/base_link.stl" scale="0.001 0.001 0.001"/>
+      <mesh filename="file://$(find cycloidal_arm)/meshes/base_link.stl" scale="0.001 0.001 0.001"/>
     </geometry>
   </collision>
 </link>
-<link name="link_1_1">
+<link name="link_1">
   <inertial>
-    <origin xyz="2.785423607376964e-17 -1.5319829840573303e-15 0.03284853130132172" rpy="0 0 0"/>
+    <origin xyz="2.785423607376964e-17 -1.5319829840573303e-15 0.03284853130132173" rpy="0 0 0"/>
     <mass value="0.6922210189689346"/>
-    <inertia ixx="0.00133" iyy="0.001397" izz="0.001299" ixy="0.0" iyz="0.0" ixz="0.0"/>
+    <inertia ixx="0.00133" iyy="0.001397" izz="0.001299" ixy="0.0" iyz="0.0" ixz="-0.0"/>
   </inertial>
   <visual>
     <origin xyz="-0.0 -0.0 -0.03" rpy="0 0 0"/>
     <geometry>
-      <mesh filename="package://cycloidal_arm/meshes/link_1_1.stl" scale="0.001 0.001 0.001"/>
+      <mesh filename="file://$(find cycloidal_arm)/meshes/link_1_1.stl" scale="0.001 0.001 0.001"/>
     </geometry>
     <material name="silver"/>
@@ -38,11 +38,11 @@
     <origin xyz="-0.0 -0.0 -0.03" rpy="0 0 0"/>
     <geometry>
-      <mesh filename="package://cycloidal_arm/meshes/link_1_1.stl" scale="0.001 0.001 0.001"/>
+      <mesh filename="file://$(find cycloidal_arm)/meshes/link_1_1.stl" scale="0.001 0.001 0.001"/>
     </geometry>
   </collision>
 </link>
-<link name="link_2_1">
+<link name="link_2">
   <inertial>
-    <origin xyz="-0.04000000000000001 -1.6058763459881033e-05 0.09471209008925147" rpy="0 0 0"/>
+    <origin xyz="-0.04 -1.6058763459882063e-05 0.09471209008925147" rpy="0 0 0"/>
     <mass value="0.7128365952218098"/>
     <inertia ixx="0.008572" iyy="0.008566" izz="0.000471" ixy="-0.0" iyz="-0.0" ixz="-0.0"/>
@@ -51,5 +51,5 @@
     <origin xyz="-0.037148 0.0 -0.14518" rpy="0 0 0"/>
     <geometry>
-      <mesh filename="package://cycloidal_arm/meshes/link_2_1.stl" scale="0.001 0.001 0.001"/>
+      <mesh filename="file://$(find cycloidal_arm)/meshes/link_2_1.stl" scale="0.001 0.001 0.001"/>
     </geometry>
     <material name="silver"/>
@@ -58,11 +58,11 @@
     <origin xyz="-0.037148 0.0 -0.14518" rpy="0 0 0"/>
     <geometry>
-      <mesh filename="package://cycloidal_arm/meshes/link_2_1.stl" scale="0.001 0.001 0.001"/>
+      <mesh filename="file://$(find cycloidal_arm)/meshes/link_2_1.stl" scale="0.001 0.001 0.001"/>
     </geometry>
   </collision>
 </link>
-<link name="link_3_1">
+<link name="link_3">
   <inertial>
-    <origin xyz="-0.03999979461983164 -4.10877760374522e-06 0.036295042070174754" rpy="0 0 0"/>
+    <origin xyz="-0.03999979461983164 -4.10877760374872e-06 0.036295042070174754" rpy="0 0 0"/>
     <mass value="0.5220823279917146"/>
     <inertia ixx="0.001597" iyy="0.001522" izz="0.000285" ixy="-0.0" iyz="0.0" ixz="-0.0"/>
@@ -71,5 +71,5 @@
     <origin xyz="-0.034338 -0.0 -0.446144" rpy="0 0 0"/>
     <geometry>
-      <mesh filename="package://cycloidal_arm/meshes/link_3_1.stl" scale="0.001 0.001 0.001"/>
+      <mesh filename="file://$(find cycloidal_arm)/meshes/link_3_1.stl" scale="0.001 0.001 0.001"/>
     </geometry>
     <material name="silver"/>
@@ -78,12 +78,12 @@
     <origin xyz="-0.034338 -0.0 -0.446144" rpy="0 0 0"/>
     <geometry>
-      <mesh filename="package://cycloidal_arm/meshes/link_3_1.stl" scale="0.001 0.001 0.001"/>
+      <mesh filename="file://$(find cycloidal_arm)/meshes/link_3_1.stl" scale="0.001 0.001 0.001"/>
     </geometry>
   </collision>
 </link>
-<link name="link_4_1">
+<link name="link_4">
   <inertial>
-    <origin xyz="2.0572304345115033e-07 -1.862792863760201e-10 0.02013378523502929" rpy="0 0 0"/>
-    <mass value="0.0712412387691247"/>
+    <origin xyz="2.057230434589566e-07 -1.8627928064288893e-10 0.024133785235029404" rpy="0 0 0"/>
+    <mass value="0.07124123876912478"/>
     <inertia ixx="5e-05" iyy="0.000214" izz="0.000193" ixy="-0.0" iyz="0.0" ixz="-0.0"/>
   </inertial>
@@ -91,5 +91,5 @@
     <origin xyz="0.005662 0.0 -0.611106" rpy="0 0 0"/>
     <geometry>
-      <mesh filename="package://cycloidal_arm/meshes/link_4_1.stl" scale="0.001 0.001 0.001"/>
+      <mesh filename="file://$(find cycloidal_arm)/meshes/link_4_1.stl" scale="0.001 0.001 0.001"/>
     </geometry>
     <material name="silver"/>
@@ -98,84 +98,88 @@
     <origin xyz="0.005662 0.0 -0.611106" rpy="0 0 0"/>
     <geometry>
-      <mesh filename="package://cycloidal_arm/meshes/link_4_1.stl" scale="0.001 0.001 0.001"/>
+      <mesh filename="file://$(find cycloidal_arm)/meshes/link_4_1.stl" scale="0.001 0.001 0.001"/>
     </geometry>
   </collision>
 </link>
-<link name="link_5_1">
+<link name="link_5">
   <inertial>
-    <origin xyz="-0.05999979427694806 -1.8626450485028255e-10 1.6900727961566275e-07" rpy="0 0 0"/>
+    <origin xyz="-0.05999979427694806 -1.8626450962614486e-10 1.6900727983770736e-07" rpy="0 0 0"/>
     <mass value="0.16139766351321969"/>
-    <inertia ixx="8e-05" iyy="0.000145" izz="0.000214" ixy="0.0" iyz="0.0" ixz="0.0"/>
+    <inertia ixx="8e-05" iyy="0.000145" izz="0.000214" ixy="0.0" iyz="-0.0" ixz="0.0"/>
   </inertial>
   <visual>
-    <origin xyz="-0.054338 0.0 -0.657106" rpy="0 0 0"/>
+    <origin xyz="-0.054338 0.0 -0.661106" rpy="0 0 0"/>
     <geometry>
-      <mesh filename="package://cycloidal_arm/meshes/link_5_1.stl" scale="0.001 0.001 0.001"/>
+      <mesh filename="file://$(find cycloidal_arm)/meshes/link_5_1.stl" scale="0.001 0.001 0.001"/>
     </geometry>
     <material name="silver"/>
   </visual>
   <collision>
-    <origin xyz="-0.054338 0.0 -0.657106" rpy="0 0 0"/>
+    <origin xyz="-0.054338 0.0 -0.661106" rpy="0 0 0"/>
     <geometry>
-      <mesh filename="package://cycloidal_arm/meshes/link_5_1.stl" scale="0.001 0.001 0.001"/>
+      <mesh filename="file://$(find cycloidal_arm)/meshes/link_5_1.stl" scale="0.001 0.001 0.001"/>
     </geometry>
   </collision>
 </link>
-<link name="camera_1">
+<link name="camera">
   <inertial>
-    <origin xyz="2.0572305194262175e-07 -1.8626450639658287e-10 0.010000169005066062" rpy="0 0 0"/>
+    <origin xyz="2.0572305194262175e-07 -1.8626450660050708e-10 0.010000169005066173" rpy="0 0 0"/>
     <mass value="0.301"/>
-    <inertia ixx="7.3e-05" iyy="7.3e-05" izz="0.000125" ixy="0.0" iyz="-0.0" ixz="-0.0"/>
+    <inertia ixx="7.3e-05" iyy="7.3e-05" izz="0.000125" ixy="0.0" iyz="0.0" ixz="0.0"/>
   </inertial>
   <visual>
-    <origin xyz="0.005662 0.0 -0.667106" rpy="0 0 0"/>
+    <origin xyz="0.005662 0.0 -0.671106" rpy="0 0 0"/>
     <geometry>
-      <mesh filename="package://cycloidal_arm/meshes/camera_1.stl" scale="0.001 0.001 0.001"/>
+      <mesh filename="file://$(find cycloidal_arm)/meshes/camera_1.stl" scale="0.001 0.001 0.001"/>
     </geometry>
     <material name="silver"/>
   </visual>
   <collision>
-    <origin xyz="0.005662 0.0 -0.667106" rpy="0 0 0"/>
+    <origin xyz="0.005662 0.0 -0.671106" rpy="0 0 0"/>
     <geometry>
-      <mesh filename="package://cycloidal_arm/meshes/camera_1.stl" scale="0.001 0.001 0.001"/>
+      <mesh filename="file://$(find cycloidal_arm)/meshes/camera_1.stl" scale="0.001 0.001 0.001"/>
     </geometry>
   </collision>
 </link>
-<joint name="Revolute_1" type="continuous">
+<joint name="Revolute_1" type="revolute">
   <origin xyz="0.0 0.0 0.03" rpy="0 0 0"/>
   <parent link="base_link"/>
-  <child link="link_1_1"/>
+  <child link="link_1"/>
   <axis xyz="0.0 0.0 1.0"/>
+  <limit upper="2.268928" lower="-2.268928" effort="100" velocity="100"/>
 </joint>
-<joint name="Revolute_2" type="continuous">
+<joint name="Revolute_2" type="revolute">
   <origin xyz="0.037148 -0.0 0.11518" rpy="0 0 0"/>
-  <parent link="link_1_1"/>
-  <child link="link_2_1"/>
+  <parent link="link_1"/>
+  <child link="link_2"/>
   <axis xyz="-1.0 0.0 0.0"/>
+  <limit upper="1.570796" lower="-1.570796" effort="100" velocity="100"/>
 </joint>
-<joint name="Revolute_3" type="continuous">
+<joint name="Revolute_3" type="revolute">
   <origin xyz="-0.00281 0.0 0.300964" rpy="0 0 0"/>
-  <parent link="link_2_1"/>
-  <child link="link_3_1"/>
-  <axis xyz="1.0 0.0 0.0"/>
+  <parent link="link_2"/>
+  <child link="link_3"/>
+  <axis xyz="-1.0 0.0 0.0"/>
+  <limit upper="1.570796" lower="-1.570796" effort="100" velocity="100"/>
 </joint>
 <joint name="Revolute_4" type="continuous">
   <origin xyz="-0.04 -0.0 0.164962" rpy="0 0 0"/>
-  <parent link="link_3_1"/>
-  <child link="link_4_1"/>
+  <parent link="link_3"/>
+  <child link="link_4"/>
   <axis xyz="0.0 0.0 1.0"/>
 </joint>
-<joint name="Revolute_5" type="continuous">
-  <origin xyz="0.06 0.0 0.046" rpy="0 0 0"/>
-  <parent link="link_4_1"/>
-  <child link="link_5_1"/>
+<joint name="Revolute_5" type="revolute">
+  <origin xyz="0.06 0.0 0.05" rpy="0 0 0"/>
+  <parent link="link_4"/>
+  <child link="link_5"/>
   <axis xyz="-1.0 0.0 0.0"/>
+  <limit upper="1.570796" lower="-1.570796" effort="100" velocity="100"/>
 </joint>
-<joint name="Rigid 6" type="fixed">
+<joint name="camera_joint" type="fixed">
   <origin xyz="-0.06 0.0 0.01" rpy="0 0 0"/>
-  <parent link="link_5_1"/>
-  <child link="camera_1"/>
+  <parent link="link_5"/>
+  <child link="camera"/>
 </joint>
-<xacro:include filename="$(find cycloidal_arm)/urdf/arm_trans.xacro" />
-<xacro:include filename="$(find cycloidal_arm)/urdf/arm_controller.xacro" />
+<!-- <xacro:include filename="$(find cycloidal_arm)/urdf/cycloidal_arm.trans" /> -->
+<xacro:include filename="$(find cycloidal_arm)/urdf/arm_gazebo.xacro" />
 </robot>
